File: firmware/Learning/storage.kicad_sch (KiCad schematic)
At the start: 0 parts

Commit message: base connections for mainboard reference
Other:
- note added: "Incoming data: 70-byte packets at 50 Hz = 3.5 kB/s nominal. Allow additional protocol and logging overhead, plus growth margin. Target storage capacity: 1 Gbit. Recover completed records after interrupted writes."
- note removed: "Sustained payload target: 7.5 MB/s, pending confirmation. Capacity and recording duration: TBD. Recover completed records after interrupted writes."
Changed lines of the file:
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@@
 	(generator_version "10.0")
 	(paper "A4")
-	(text "Sustained payload target: 7.5 MB/s, pending confirmation. Capacity and recording duration: TBD. Recover completed records after interrupted writes."
+	(text "Incoming data: 70-byte packets at 50 Hz = 3.5 kB/s nominal. Allow additional protocol and logging overhead, plus growth margin.\nTarget storage capacity: 1 Gbit.\nRecover completed records after interrupted writes."
 		(exclude_from_sim no)
-		(at 100.076 14.986 0)
+		(at 97.282 17.78 0)
 		(effects
 			(font
